File: Hardware/Buzzer Box/Spannungswandler.kicad_sch (KiCad schematic)
At the start: 3 parts

Commit message: made chages to the PCB
Other:
- company: (none) -> EinfachTechnik
- title: (none) -> BuzzerPCB
Changed lines of the file:
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@@
 	(generator_version "8.0")
 	(paper "A4")
+	(title_block
+		(title "BuzzerPCB")
+		(date "2024-12-23")
+		(rev "2")
+		(company "EinfachTechnik")
+	)
 	(junction
 		(at 114.3 109.22)
